File: hardware/beat.kicad_pcb (KiCad board)
At the start: 4 copper layers, 60 x 35 mm, 68 parts, among them J101 Cortex_Debug, J102 JAE_DX07S016JA3, J103 Output, J601 SJ2-25404B-SMT-TR, Q201 IQE006NE2LM5CGSC, Q301 IQE006NE2LM5CGSC, Q401 IQE006NE2LM5CGSC, Q501 IQE006NE2LM5CGSC, SW101 SW_Push, SW102 SW_Push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

Commit message: Refresh
Parts:
- removed the C102 at (148.5, 93.2)
- added ?: , clipboard:c642ec12-5240-48df-bbfd-b5e940fbc8ac, F.Cu at (133.2, 108.8)
- added ?: , clipboard:c642ec12-5240-48df-bbfd-b5e940fbc8ac, F.Cu at (133.2, 109.2)
- C101, C201, C301, C401, C501, C601, C602: footprint Capacitor_SMD:C_0603_1608Metric -> V2_Capacitor_SMD:C_0603
- C102: renamed from C103; footprint Capacitor_SMD:C_0603_1608Metric -> V2_Capacitor_SMD:C_0603
- C103: renamed from C104; footprint Capacitor_SMD:C_0603_1608Metric -> V2_Capacitor_SMD:C_0603
- C104: renamed from C105; footprint Capacitor_SMD:C_0603_1608Metric -> V2_Capacitor_SMD:C_0603
- C105: renamed from C106; footprint Capacitor_SMD:C_0603_1608Metric -> V2_Capacitor_SMD:C_0603
- C106: renamed from C107; footprint Capacitor_SMD:C_0603_1608Metric -> V2_Capacitor_SMD:C_0805
- C107: renamed from C108; footprint Capacitor_SMD:C_0603_1608Metric -> V2_Capacitor_SMD:C_0805
- C108: renamed from C109; footprint Capacitor_SMD:C_0603_1608Metric -> V2_Capacitor_SMD:C_0603
- C109: renamed from C110; footprint Capacitor_SMD:C_0603_1608Metric -> V2_Capacitor_SMD:C_0603
- C110: renamed from C111; footprint Capacitor_SMD:C_1210_3225Metric -> V2_Capacitor_SMD:C_1210
- C111: renamed from C112; footprint Capacitor_SMD:C_0603_1608Metric -> V2_Capacitor_SMD:C_0603
- C112: renamed from C113; footprint Capacitor_SMD:C_0603_1608Metric -> V2_Capacitor_SMD:C_0603
- D103: footprint LED_SMD:LED_0603_1608Metric -> V2_LED:LED_0603
- D104, D601: footprint Diode_SMD:D_SOD-523 -> V2_Diode_SMD:D_SOD-523
- D201, D301, D401, D501: footprint Diode_SMD:D_SOD-123F -> V2_Diode_SMD:D_SOD-123F
- FID101, FID102, FID103: value Fiducial -> Fiducial_Paste
- INFO102: value ORDER-NUMBER -> Order_Number
- J102: value JAE_DX07S016JA3 -> DX07S016JA3
- J103: value Output -> ~
- Q201, Q301, Q401, Q501: value IQE006NE2LM5CGSC -> IQE022N06LM5CGSCATMA1
- R101, R102, R103, R104, R105, R601, R701: footprint Resistor_SMD:R_0603_1608Metric -> V2_Resistor_SMD:R_0603
- SW101, SW102: value SW_Push -> SKSG
- TVS101: footprint Diode_SMD:D_0603_1608Metric -> V2_Diode_SMD:D_0603
- U601: footprint Package_SO:SO-5-6_4.55x3.7mm_P1.27mm -> V2_Package_SO:SO-5-6_4.55x3.7mm_P1.27mm
- moved INFO101 59.0 mm to (124.5, 81.0), turned to 180 degrees
- moved ESD101 1.68 mm to (131.5, 106.5)
- moved C101 1.03 mm to (148.8, 92.8), turned to 180 degrees
- moved C103 1.00 mm to (145.8, 92.8), turned to 0 degrees
- moved C105 0.56 mm to (141.2, 99.5)
- moved C106 0.25 mm to (136.2, 110.2)
- moved C107 0.25 mm to (136.2, 103.8)
- moved TVS101 0.25 mm to (136.2, 112.2)
Connections:
- net USB-Shield renamed Shield
Routing:
- net +3V3: track 24.7 -> 90.5 mm
- net /LED1: track 26.3 -> 45.4 mm
- net /+5V-PWM: track 34.6 -> 23.0 mm
- net /USB-: track 38.2 -> 45.3 mm, vias 3 -> 4
- net /Fault: track 28.0 -> 21.5 mm
- net /USB+: track 36.5 -> 42.6 mm, vias 3 -> 2
- net GND: track 30.6 -> 34.8 mm, vias 71 -> 98
- net +5V: track 49.8 -> 51.7 mm
- net /PWM3: track 21.9 -> 22.5 mm
- net /USB-CC1: track 5.39 -> 5.89 mm
- added copper zone on B.Cu, net +5V
- removed copper zone on In2.Cu, net +3V3
- removed copper zone on In2.Cu, net +5V
- removed copper zone on B.Cu, net GND

Commit message: Update
Parts:
- removed ? (x2): , clipboard:c642ec12-5240-48df-bbfd-b5e940fbc8ac
- moved D103 1.25 mm to (153.2, 93.0)
- moved R101 1.25 mm to (153.2, 91.5)
- moved R104 1.25 mm to (153.2, 90.0)
- moved C102 0.79 mm to (152.5, 95.5), turned to -90 degrees
Routing:
- net GND: track 34.8 -> 36.2 mm
- net /USB-: track 45.3 -> 44.6 mm
- net +3V3: track 90.5 -> 89.9 mm
- net /LED-onboard: track 4.40 -> 4.94 mm

Commit message: Refresh
Parts:
- J103: value ~ -> 1x08
- Q201, Q301, Q401, Q501: value IQE022N06LM5CGSCATMA1 -> IQE006NE2LM5CGSC

Commit message: Update library
Parts:
- J101: footprint V2_Cortex_Debug:Cortex_Debug_Pad -> V2_Connector_Debug:Cortex
- Q201, Q301, Q401, Q501: value IQE006NE2LM5CGSC -> IQE006NE2LM5CG
Routing:
- net GND: vias 98 -> 96
- net +3V3: vias 11 -> 10
