File: hardware/beat.kicad_pcb (KiCad board)
At the start: 4 copper layers, 60 x 35 mm, 67 parts, among them J101 Cortex, J102 1x08, J103 DX07S016JA3, J601 SJ2-25404B-SMT-TR, Q201 IQE006NE2LM5CG, Q301 IQE006NE2LM5CG, Q401 IQE006NE2LM5CG, Q501 IQE006NE2LM5CG, SW101 SKSG, SW102 SKSG, U101 ATSAMD51G, U102 TPS78433QWDRBRQ1, U601 TLP2361, U701 TPS2559, Y101 32k768

Commit message: Refresh
Parts:
- C101, C102, C103, C104, C105, C106, C107, C108, C109, C201, C301, C401, C501, C601, C602: footprint V2_Capacitor_SMD:C_0603 -> V2_Capacitor_SMD:C_1608
- C110, C111: footprint V2_Capacitor_SMD:C_0805 -> V2_Capacitor_SMD:C_2012
- C112: footprint V2_Capacitor_SMD:C_1210 -> V2_Capacitor_SMD:C_3225
- D102: footprint V2_LED:LED_0603 -> V2_LED:LED_1608
- INFO102: value Layer_Numbers -> Layer_Numbers-4; footprint V2_Production:Layer_Numbers -> V2_Production:Layer_Numbers-4
- R101, R102, R103, R104, R105, R601, R701: footprint V2_Resistor_SMD:R_0603 -> V2_Resistor_SMD:R_1608
- TVS101: footprint V2_Diode_SMD:D_0603 -> V2_Diode_SMD:D_1608
Routing:
- net +5V: track 52.0 -> 50.2 mm
- net /Resistance-Sense: track 22.0 -> 20.5 mm
- net /MIDI In/Tip: track 20.0 -> 21.4 mm
- net GND: vias 96 -> 97
