File: hardware/beat.kicad_pcb (KiCad board)
At the start: 4 copper layers, 60 x 35 mm, 67 parts, among them J101 Cortex, J102 1x08, J103 DX07S016JA3, J601 SJ2-25404B-SMT-TR, Q201 IQE006NE2LM5CG, Q301 IQE006NE2LM5CG, Q401 IQE006NE2LM5CG, Q501 IQE006NE2LM5CG, SW101 SKSG, SW102 SKSG, U101 ATSAMD51G, U102 TPS78433QWDRBRQ1, U601 TLP2361, U701 TPS2559, Y101 32k768

Commit message: Add front + back
Connections:
- ESD101 pad 2: unconnected-(ESD101-D2-Pad2) -> /USB-
- ESD101 pad 3: unconnected-(ESD101-D1-Pad3) -> /USB+
Routing:
- net /USB+: track 42.5 -> 41.3 mm
- net /USB-: track 44.4 -> 44.1 mm, vias 4 -> 2
Other:
- outline, holes or cut-outs redrawn

Commit message: Refresh
Connections:
- net /+5V-PWM renamed /+VPWM
- net /PWMOut1 renamed /PWM-Sink-1
- net /PWMOut2 renamed /PWM-Sink-2
- net /PWMOut3 renamed /PWM-Sink-3
- net /PWMOut4 renamed /PWM-Sink-4
- U102 pad 6: unconnected-(U102-Pad6) -> +5V
