File: hardware/beat.kicad_sch (KiCad schematic)
At the start: 44 parts, among them J101 Cortex_Debug, J102 JAE_DX07S016JA3, J103 Output, SW101 SW_Push, SW102 SW_Push, U101 TPS78433QWDRBRQ1, U102 ATSAMD51G, Y101 32k768

Commit message: Refresh
Parts:
- removed C102: 0u1, Capacitor_SMD:C_0603_1608Metric, symbol Device:C_Small
- C101: footprint Capacitor_SMD:C_0603_1608Metric -> V2_Capacitor_SMD:C_0603; symbol Device:C_Small -> V2_Device:C_0603_10u; Manufacturer (none) -> TDK; Mouser (none) -> 810-C1608X6S1A106M; Product (none) -> C1608X6S1A106M080AC
- C102: renamed from C103; footprint Capacitor_SMD:C_0603_1608Metric -> V2_Capacitor_SMD:C_0603; symbol Device:C_Small -> V2_Device:C_0603_0u1; Manufacturer (none) -> TDK; Mouser (none) -> 810-CGA3E2X7R1H104MA; Product (none) -> CGA3E2X7R1H104M080AA
- C103: renamed from C104; footprint Capacitor_SMD:C_0603_1608Metric -> V2_Capacitor_SMD:C_0603; symbol Device:C_Small -> V2_Device:C_0603_0u1; Manufacturer (none) -> TDK; Mouser (none) -> 810-CGA3E2X7R1H104MA; Product (none) -> CGA3E2X7R1H104M080AA
- C104: renamed from C105; footprint Capacitor_SMD:C_0603_1608Metric -> V2_Capacitor_SMD:C_0603; symbol Device:C_Small -> V2_Device:C_0603_0u1; Manufacturer (none) -> TDK; Mouser (none) -> 810-CGA3E2X7R1H104MA; Product (none) -> CGA3E2X7R1H104M080AA
- C105: renamed from C106; footprint Capacitor_SMD:C_0603_1608Metric -> V2_Capacitor_SMD:C_0603; symbol Device:C_Small -> V2_Device:C_0603_0u1; Manufacturer (none) -> TDK; Mouser (none) -> 810-CGA3E2X7R1H104MA; Product (none) -> CGA3E2X7R1H104M080AA
- C106: renamed from C107; footprint Capacitor_SMD:C_0603_1608Metric -> V2_Capacitor_SMD:C_0805; symbol Device:C_Small -> V2_Device:C_0805_10u; Manufacturer (none) -> TDK; Mouser (none) -> 810-C2012X5R1E106K; Product (none) -> C2012X5R1E106K125AB; Rating (none) -> 25V
- C107: renamed from C108; footprint Capacitor_SMD:C_0603_1608Metric -> V2_Capacitor_SMD:C_0805; symbol Device:C_Small -> V2_Device:C_0805_10u; Manufacturer (none) -> TDK; Mouser (none) -> 810-C2012X5R1E106K; Product (none) -> C2012X5R1E106K125AB; Rating (none) -> 25V
- C108: renamed from C109; footprint Capacitor_SMD:C_0603_1608Metric -> V2_Capacitor_SMD:C_0603; symbol Device:C_Small -> V2_Device:C_0603_18p; Manufacturer (none) -> YAGEO; Mouser (none) -> 603-CC603JRNPO9BN180; Product (none) -> CC0603JRNPO9BN180
- C109: renamed from C110; footprint Capacitor_SMD:C_0603_1608Metric -> V2_Capacitor_SMD:C_0603; symbol Device:C_Small -> V2_Device:C_0603_18p; Manufacturer (none) -> YAGEO; Mouser (none) -> 603-CC603JRNPO9BN180; Product (none) -> CC0603JRNPO9BN180
- C110: renamed from C111; footprint Capacitor_SMD:C_1210_3225Metric -> V2_Capacitor_SMD:C_1210; symbol Device:C_Small -> V2_Device:C_1210_22u; Manufacturer (none) -> TDK; Mouser (none) -> 810-CGA6P3X7R1E226M5; Product (none) -> CGA6P3X7R1E226M250AE; Voltage (none) -> 25V
- C111: renamed from C112; footprint Capacitor_SMD:C_0603_1608Metric -> V2_Capacitor_SMD:C_0603; symbol Device:C_Small -> V2_Device:C_0603_0u1; Manufacturer (none) -> TDK; Mouser (none) -> 810-CGA3E2X7R1H104MA; Product (none) -> CGA3E2X7R1H104M080AA
- C112: renamed from C113; footprint Capacitor_SMD:C_0603_1608Metric -> V2_Capacitor_SMD:C_0603; symbol Device:C_Small -> V2_Device:C_0603_0u1; Manufacturer (none) -> TDK; Mouser (none) -> 810-CGA3E2X7R1H104MA; Product (none) -> CGA3E2X7R1H104M080AA
- D101, D102: LCSC (none) -> C965555; Manufacturer (none) -> Worldsemi; Product (none) -> WS2812B-2020
- D103: footprint LED_SMD:LED_0603_1608Metric -> V2_LED:LED_0603; symbol Device:LED_Small -> V2_Device:LED_0603_Orange; Manufacturer (none) -> ROHM Semiconductor; Mouser (none) -> 755-SML-D12M8WT86C; Product (none) -> SML-D12M8WT86C
- D104: footprint Diode_SMD:D_SOD-523 -> V2_Diode_SMD:D_SOD-523; Manufacturer (none) -> ROHM Semiconductor; Mouser (none) -> 755-RB501SM-30FHT2R; Product (none) -> RB501SM-30FHT2R
- ESD101: Manufacturer (none) -> Semtech; Mouser (none) -> 947-RCLAMP0582N.TCT; Product (none) -> RCLAMP0582N.TCT
- FID101, FID102, FID103: value Fiducial -> Fiducial_Paste
- INFO102: value ORDER-NUMBER -> Order_Number
- J102: value JAE_DX07S016JA3 -> DX07S016JA3; Manufacturer (none) -> JAE Electronics; Mouser (none) -> 656-DX07S016JA3R1500; Product (none) -> DX07S016JA3R1500
- J103: value Output -> ~
- R101: footprint Resistor_SMD:R_0603_1608Metric -> V2_Resistor_SMD:R_0603; symbol Device:R_Small -> V2_Device:R_0603_330R; Manufacturer (none) -> Vishay; Mouser (none) -> 71-CRCW0603330RFKEAC; Product (none) -> CRCW0603330RFKEAC; Rating (none) -> 100mW
- R102, R103: footprint Resistor_SMD:R_0603_1608Metric -> V2_Resistor_SMD:R_0603; symbol Device:R_Small -> V2_Device:R_0603_5k1; Manufacturer (none) -> Vishay; Mouser (none) -> 71-CRCW06035K10FKEAC; Product (none) -> CRCW06035K10FKEAC; Rating (none) -> 100mW
- R104: footprint Resistor_SMD:R_0603_1608Metric -> V2_Resistor_SMD:R_0603; symbol Device:R_Small -> V2_Device:R_0603_100k; Manufacturer (none) -> Vishay; Mouser (none) -> 71-CRCW0603100KFKEAC; Product (none) -> CRCW0603100KFKEAC; Rating (none) -> 100mW
- R105: footprint Resistor_SMD:R_0603_1608Metric -> V2_Resistor_SMD:R_0603; symbol Device:R_Small -> V2_Device:R_0603_100R; Manufacturer (none) -> Vishay; Mouser (none) -> 71-CRCW0603100RFKEAH; Product (none) -> CRCW0603100RFKEAHP; Rating (none) -> 330mW
- SW101, SW102: value SW_Push -> SKSG; symbol Switch:SW_Push -> V2_Switch:SKSG; Manufacturer (none) -> Alps Alpine; Mouser (none) -> 688-SKSGACE010; Product (none) -> SKSGACE010
- TVS101: footprint Diode_SMD:D_0603_1608Metric -> V2_Diode_SMD:D_0603; Manufacturer (none) -> Bourns; Mouser (none) -> 652-CG0603MLC-05LE; Product (none) -> CG0603MLC-05LE; Rating (none) -> 5V
- U101: Manufacturer (none) -> Texas Instruments; Mouser (none) -> 595-TPS78433QWDRBRQ1; Product (none) -> TPS78433QWDRBRQ1
- U102: Manufacturer (none) -> Microchip Technology; Mouser (none) -> 556-ATSAMD51G19AMU; Product (none) -> ATSAMD51G19A-MU
- Y101: symbol Device:Crystal_Small -> V2_Device:Crystal_3.2x1.5_32k768; Manufacturer (none) -> ABRACON; Mouser (none) -> 815-ABS0716632.768KT; Product (none) -> ABS07-166-32.768KHZ-T
Connections:
- net USB-Shield renamed Shield
Other:
- note added: "100R / Solenoid coil voltage divider Supplies reference voltage to a single channel while the +24V power is switched off."
- note removed: "100R / Solenoid coil voltage divider to measure the solenoid resistance. Supplies a reference voltage to a single channel while the power is switched off."
- moved on the sheet: C101, C106, C107, C110, ICON101, ICON102, INFO102, J103, U101

Commit message: Update
Parts:
- J103: value ~ -> 1x08
Changed lines of the file:
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@@
 			)
 		)
-		(property "Value" "~"
+		(property "Value" "1x08"
 			(at 156.21 157.48 0)
 			(effects

Commit message: Refresh
Parts:
- D103: Mouser 755-SML-D12M8WT86C -> 755-SML-D12D1WT86; Product SML-D12M8WT86C -> SML-D12D1WT86

Commit message: Update library
Parts:
- C101: Rating (none) -> 10V
- C102, C103, C104, C105, C111, C112: Rating (none) -> 50V
- C110: Rating (none) -> 25V; Voltage 25V -> (none)
- J101: footprint V2_Cortex_Debug:Cortex_Debug_Pad -> V2_Connector_Debug:Cortex; symbol V2_Cortex_Debug:Cortex_Debug -> V2_Connector_Debug:Cortex

Commit message: Replace Order_Number
Parts:
- H101, H102, H103, H104: value MountingHole_2mm -> 2mm
- INFO102: value Order_Number -> ~; footprint V2_Production:Order_Number -> V2_Production:Revision; symbol V2_Production:Order_Number -> V2_Production:Revision
- J101: value Cortex_Debug -> Cortex
Other:
- moved on the sheet: C110

Commit message: Update Library
Parts:
- C101: symbol V2_Device:C_0603_10u -> V2_Capacitor:0603_10u
- C102, C103, C104, C105, C111, C112: symbol V2_Device:C_0603_0u1 -> V2_Capacitor:0603_0u1
- C106, C107: symbol V2_Device:C_0805_10u -> V2_Capacitor:0805_10u
- C108, C109: symbol V2_Device:C_0603_18p -> V2_Capacitor:0603_18p
- C110: value 22u -> 10u; symbol V2_Device:C_1210_22u -> V2_Capacitor:1210_22u
- D103: symbol V2_Device:LED_0603_Orange -> V2_LED:0603_Orange
- R101: symbol V2_Device:R_0603_330R -> V2_Resistor:0603_330R
- R102, R103: symbol V2_Device:R_0603_5k1 -> V2_Resistor:0603_5k1
- R104: symbol V2_Device:R_0603_100k -> V2_Resistor:0603_100k
- R105: symbol V2_Device:R_0603_100R -> V2_Resistor:0603_100R
- Y101: symbol V2_Device:Crystal_3.2x1.5_32k768 -> V2_Crystal:3.2x1.5_32k768

Commit message: Refresh
Other:
- note added: "100R / Solenoid coil voltage divider supplies reference voltage to a single channel while the PWM power is switched off."
- note removed: "100R / Solenoid coil voltage divider Supplies reference voltage to a single channel while the +24V power is switched off."
Changed lines of the file:
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@@
 		)
 	)
-	(text "100R / Solenoid coil voltage divider\nSupplies reference voltage to a single\nchannel while the +24V power is\nswitched off."
+	(text "100R / Solenoid coil voltage divider supplies\nreference voltage to a single channel while\nthe PWM power is switched off."
 		(exclude_from_sim no)
-		(at 122.682 186.436 0)
+		(at 118.11 187.706 0)
 		(effects
 			(font
@@
 		(at 156.21 170.18 0)
 		(unit 1)
-		(exclude_from_sim no)
+		(exclude_from_sim yes)
 		(in_bom yes)
 		(on_board yes)
@@
 			)
 		)
-		(property "Sim.Enable" "0"
-			(at 156.21 170.18 0)
-			(effects
-				(font
-					(size 1.27 1.27)
-				)
-				(hide yes)
-			)
-		)
 		(pin "1"
 		)
@@
 		(at 209.55 158.115 0)
 		(unit 1)
-		(exclude_from_sim no)
+		(exclude_from_sim yes)
 		(in_bom no)
 		(on_board yes)
@@
 			)
 		)
-		(property "Sim.Enable" "0"
-			(at 209.55 158.115 0)
-			(effects
-				(font
-					(size 1.27 1.27)
-				)
-				(hide yes)
-			)
-		)
 		(instances
 			(project "beat"
@@
 		(at 181.61 172.72 0)
 		(unit 1)
-		(exclude_from_sim no)
+		(exclude_from_sim yes)
 		(in_bom no)
 		(on_board yes)
@@
 			(at 181.61 172.72 0)
 			(effects
-				(font
-					(size 1.27 1.27)
-				)
-				(hide yes)
-			)
-		)
-		(property "Sim.Enable" "0"
-			(at 181.61 172.72 0)
-			(effects
