File: hardware/beat.kicad_sch (KiCad schematic)
At the start: 43 parts, among them J101 Cortex, J102 1x08, J103 DX07S016JA3, SW101 SKSG, SW102 SKSG, U101 ATSAMD51G, U102 TPS78433QWDRBRQ1, Y101 32k768

Commit message: Refresh
Parts:
- D102: footprint V2_LED:LED_0603 -> V2_LED:LED_1608
- INFO102: value Layer_Numbers -> Layer_Numbers-4; footprint V2_Production:Layer_Numbers -> V2_Production:Layer_Numbers-4; symbol V2_Production:Layer_Numbers -> V2_Production:Layer_Numbers-4
- TVS101: footprint V2_Diode_SMD:D_0603 -> V2_Diode_SMD:D_1608

Commit message: Add front + back
Connections:
- net USB+: now also ESD101.3 (D1)
- net USB-: now also ESD101.2 (D2)
- no-connect marks 25 -> 23

Commit message: Refresh
Connections:
- net +5V: now also U102.6 (EN)
- net +5V-PWM renamed +VPWM
- net PWMOut1 renamed PWM-Sink-1
- net PWMOut2 renamed PWM-Sink-2
- net PWMOut3 renamed PWM-Sink-3
- net PWMOut4 renamed PWM-Sink-4
Other:
- sheet PWM 1 ports: added +VPWM, PWM-Sink; removed PWMOut, Power
- sheet PWM 2 ports: added +VPWM, PWM-Sink; removed PWMOut, Power
- sheet PWM 3 ports: added +VPWM, PWM-Sink; removed PWMOut, Power
- sheet PWM 4 ports: added +VPWM, PWM-Sink; removed PWMOut, Power
