File: hardware/MIDIIn.kicad_sch (KiCad schematic)
At the start: 6 parts, among them J601 SJ2-25404B-SMT-TR, U601 TLP2361

Commit message: Refresh
Parts:
- C601, C602: footprint Capacitor_SMD:C_0603_1608Metric -> V2_Capacitor_SMD:C_0603; symbol Device:C_Small -> V2_Device:C_0603_0u1; Manufacturer (none) -> TDK; Mouser (none) -> 810-CGA3E2X7R1H104MA; Product (none) -> CGA3E2X7R1H104M080AA
- D601: footprint Diode_SMD:D_SOD-523 -> V2_Diode_SMD:D_SOD-523; Manufacturer (none) -> ROHM Semiconductor; Mouser (none) -> 755-RB501SM-30FHT2R; Product (none) -> RB501SM-30FHT2R
- J601: Manufacturer (none) -> Same Sky; Mouser (none) -> 490-SJ2-25404BSMT-TR; Product (none) -> SJ2-25404B-SMT-TR
- R601: footprint Resistor_SMD:R_0603_1608Metric -> V2_Resistor_SMD:R_0603; symbol Device:R_Small -> V2_Device:R_0603_220R; Manufacturer (none) -> Vishay; Mouser (none) -> 71-CRCW0603220RFKEAH; Product (none) -> CRCW0603220RFKEAHP; Rating (none) -> 330mW
- U601: footprint Package_SO:SO-5-6_4.55x3.7mm_P1.27mm -> V2_Package_SO:SO-5-6_4.55x3.7mm_P1.27mm; Manufacturer (none) -> Toshiba; Mouser (none) -> 757-TLP2361TPRE; Product (none) -> TLP2361(TPR,E

Commit message: Update library
Parts:
- C601, C602: Rating (none) -> 50V

Commit message: Update Library
Parts:
- C601, C602: symbol V2_Device:C_0603_0u1 -> V2_Capacitor:0603_0u1
- R601: symbol V2_Device:R_0603_220R -> V2_Resistor:0603_220R

Commit message: Replace diode
Parts:
- D601: value RB501SM -> PMEG2010EPK; footprint V2_Diode_SMD:D_SOD-523 -> V2_Diode_SMD:D_SOD-1608; symbol V2_Diode:RB501SM -> V2_Diode:PMEG2010EPK; Manufacturer ROHM Semiconductor -> Nexperia; Mouser 755-RB501SM-30FHT2R -> 771-PMEG2010EPK; Product RB501SM-30FHT2R -> PMEG2010EPK; Rating (none) -> 20V
Other:
- title: MIDI In -> V2 beat
Changed lines of the file:
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@@
 (kicad_sch
-	(version 20250114)
+	(version 20260306)
 	(generator "eeschema")
-	(generator_version "9.0")
+	(generator_version "10.0")
 	(paper "A4")
 	(title_block
-		(title "MIDI In")
-		(date "2026-02-10")
-		(rev "2026-02-10")
+		(title "V2 beat")
+		(date "2026-03-30")
+		(rev "2026-03-30")
 	)

Commit message: Update
Parts:
- C601: renamed from C602; Id (none) -> Capacitor:${SYMBOL_NAME}
- C602: renamed from C601; Id (none) -> Capacitor:${SYMBOL_NAME}
- D601: Id (none) -> Diode:${SYMBOL_NAME}
- J601: Id (none) -> Audio:${SYMBOL_NAME}; Rating (none) -> 2.5mm
- R601: Id (none) -> Resistor:${SYMBOL_NAME}
- U601: Id (none) -> Optocoupler:${SYMBOL_NAME}; Rating (none) -> 15Mbps
Other:
- company: (none) -> Versio Duo
Changed lines of the file:
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@@
 	(title_block
 		(title "V2 beat")
-		(date "2026-03-30")
+		(date "2026-04-14")
 		(rev "2026-03-30")
+		(company "Versio Duo")
+		(comment 1 "Solenoid Controller")
 	)
