File: hardware/MIDIIn.kicad_sch (KiCad schematic)
At the start: 6 parts, among them J601 SJ2-25404B-SMT-TR, U601 TLP2361

Commit message: Good Bye Imperial
Parts:
- C601, C602: footprint V2_Capacitor_SMD:C_0603 -> V2_Capacitor_SMD:C_1608; symbol V2_Capacitor:0603_0u1 -> V2_Capacitor:1608_0u1
- R601: footprint V2_Resistor_SMD:R_0603 -> V2_Resistor_SMD:R_1608; symbol V2_Resistor:0603_220R -> V2_Resistor:1608_220R
