File: hardware/MIDIIn.kicad_sch (KiCad schematic)
At the start: 6 parts, among them J601 SJ2-25404B-SMT-TR, U601 TLP2361

Commit message: Refresh
Parts:
- R601: Manufacturer Vishay -> Panasonic; Mouser 71-CRCW0603220RFKEAH -> 667-ERJ-PA3F2200V; Product CRCW0603220RFKEAHP -> ERJ-PA3F2200V; Rating 330mW -> 333mW
Changed lines of the file:
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@@
 	(title_block
 		(title "V2 beat")
-		(date "2026-08-19")
+		(date "2026-08-28")
 		(rev "2026-08-19")
 		(company "Versio Duo")
