File: hardware/PowerSwitch.kicad_sch (KiCad schematic)
At the start: 2 parts, among them U701 TPS2559

Commit message: Refresh
Parts:
- R701: footprint Resistor_SMD:R_0603_1608Metric -> V2_Resistor_SMD:R_0603; symbol Device:R_Small -> V2_Device:R_0603_39k; Manufacturer (none) -> Vishay; Mouser (none) -> 71-RCS060339K0FKEA; Product (none) -> RCS060339K0FKEA; Rating (none) -> 500mW
- U701: Manufacturer (none) -> Texas Instruments; Mouser (none) -> 595-TPS2559DRCR; Product (none) -> TPS2559DRCR
Changed lines of the file:
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@@
 	)
 	(symbol
-		(lib_id "power:+5V")
+		(lib_id "V2_power:+5V")
 		(at 146.05 99.06 90)
 		(unit 1)
@@
 	)
 	(symbol
-		(lib_id "power:GND")
+		(lib_id "V2_power:GND")
 		(at 133.35 114.3 270)
 		(unit 1)
@@
 			)
 		)
+		(property "Mouser" "595-TPS2559DRCR"
+			(at 156.21 132.08 0)
+			(effects
+				(font
+					(size 1.27 1.27)
+				)
+				(hide yes)
+			)
+		)
+		(property "Product" "TPS2559DRCR"
+			(at 156.21 129.54 0)
+			(effects
+				(font
+					(size 1.27 1.27)
+				)
+				(hide yes)
+			)
+		)
+		(property "Manufacturer" "Texas Instruments"
+			(at 156.21 127 0)
+			(effects
+				(font
+					(size 1.27 1.27)
+				)
+				(hide yes)
+			)
+		)
+		(property "Sim.Pin" ""
+			(at 156.21 106.68 0)
+			(effects
+				(font
+					(size 1.27 1.27)
+				)
+				(hide yes)
+			)
+		)
 		(pin "1"
 		)
@@
 	)
 	(symbol
-		(lib_id "Device:R_Small")
+		(lib_id "V2_Device:R_0603_39k")
 		(at 135.89 114.3 270)
 		(unit 1)
@@
 			)
 		)
-		(property "Footprint" "Resistor_SMD:R_0603_1608Metric"
+		(property "Footprint" "V2_Resistor_SMD:R_0603"
+			(at 120.142 114.3 0)
+			(effects
+				(font
+					(size 1.27 1.27)
+				)
+				(hide yes)
+			)
+		)
+		(property "Datasheet" ""
 			(at 135.89 114.3 0)
 			(effects
@@
 			)
 		)
-		(property "Datasheet" "~"
-			(at 135.89 114.3 0)
-			(effects
-				(font
-					(size 1.27 1.27)
-				)
-				(hide yes)
-			)
-		)
 		(property "Description" "Resistor, small symbol"
-			(at 135.89 114.3 0)
+			(at 123.19 114.3 0)
+			(effects
+				(font
+					(size 1.27 1.27)
+				)
+				(hide yes)
+			)
+		)
+		(property "Mouser" "71-RCS060339K0FKEA"
+			(at 113.03 114.3 0)
+			(effects
+				(font
+					(size 1.27 1.27)
+				)
+				(hide yes)
+			)
+		)
+		(property "Rating" "500mW"
+			(at 115.57 114.3 0)
+			(effects
+				(font
+					(size 1.27 1.27)
+				)
+				(hide yes)
+			)
+		)
+		(property "Manufacturer" "Vishay"
+			(at 120.65 114.3 0)
+			(effects
+				(font
+					(size 1.27 1.27)
+				)
+				(hide yes)
+			)
+		)
+		(property "Product" "RCS060339K0FKEA"
+			(at 118.11 114.3 0)
+			(effects
+				(font
+					(size 1.27 1.27)
+				)
+				(hide yes)
+			)
+		)
+		(property "Sim.Pin" ""
+			(at 135.89 114.3 90)
 			(effects
 				(font
@@
 	)
 	(symbol
-		(lib_id "power:GND")
+		(lib_id "V2_power:GND")
 		(at 166.37 114.3 90)
 		(unit 1)

Commit message: Update Library
Parts:
- R701: symbol V2_Device:R_0603_39k -> V2_Resistor:0603_39k
Changed lines of the file:
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@@
 		(on_board yes)
 		(dnp no)
-		(property "Reference" "#PWR0701"
+		(property "Reference" "#PWR701"
 			(at 149.86 99.06 0)
 			(effects
@@
 			(project "beat"
 				(path "/6c8448b4-b04d-47e1-934e-e40cbe27a7be/0ac9d349-3066-4d6a-93e7-4d57eaae463a"
-					(reference "#PWR0701")
+					(reference "#PWR701")
 					(unit 1)
 				)
@@
 		(dnp no)
 		(fields_autoplaced yes)
-		(property "Reference" "#PWR0702"
+		(property "Reference" "#PWR702"
 			(at 127 114.3 0)
 			(effects
@@
 			(project "beat"
 				(path "/6c8448b4-b04d-47e1-934e-e40cbe27a7be/0ac9d349-3066-4d6a-93e7-4d57eaae463a"
-					(reference "#PWR0702")
+					(reference "#PWR702")
 					(unit 1)
 				)
@@
 	)
 	(symbol
-		(lib_id "V2_Device:R_0603_39k")
+		(lib_id "V2_Resistor:0603_39k")
 		(at 135.89 114.3 270)
 		(unit 1)
@@
 		(dnp no)
 		(fields_autoplaced yes)
-		(property "Reference" "#PWR0703"
+		(property "Reference" "#PWR703"
 			(at 172.72 114.3 0)
 			(effects
@@
 			(project "beat"
 				(path "/6c8448b4-b04d-47e1-934e-e40cbe27a7be/0ac9d349-3066-4d6a-93e7-4d57eaae463a"
-					(reference "#PWR0703")
-					(unit 1)
-				)
+					(reference "#PWR703")
+					(unit 1)
+				)

Commit message: Replace diode
Other:
- title: Power Switch 5V -> V2 beat

Commit message: Update
Parts:
- R701: Id (none) -> Resistor:${SYMBOL_NAME}
- U701: Id (none) -> PowerSwitch:${SYMBOL_NAME}; Rating (none) -> 4.7A
Changed lines of the file:
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@@
 	(title_block
 		(title "V2 beat")
-		(date "2026-03-30")
+		(date "2026-04-14")
 		(rev "2026-03-30")
 		(company "Versio Duo")
+		(comment 1 "Solenoid Controller")
 	)
 	(rectangle
@@
 		(in_pos_files yes)
 		(dnp no)
-		(property "Reference" "#PWR701"
+		(property "Reference" "#PWR0702"
 			(at 149.86 99.06 0)
 			(hide yes)
@@
 			(project "beat"
 				(path "/6c8448b4-b04d-47e1-934e-e40cbe27a7be/0ac9d349-3066-4d6a-93e7-4d57eaae463a"
-					(reference "#PWR701")
+					(reference "#PWR0702")
 					(unit 1)
 				)
@@
 		(dnp no)
 		(fields_autoplaced yes)
-		(property "Reference" "#PWR702"
+		(property "Reference" "#PWR0701"
 			(at 127 114.3 0)
 			(hide yes)
@@
 			(project "beat"
 				(path "/6c8448b4-b04d-47e1-934e-e40cbe27a7be/0ac9d349-3066-4d6a-93e7-4d57eaae463a"
-					(reference "#PWR702")
+					(reference "#PWR0701")
 					(unit 1)
 				)
@@
 			)
 		)
+		(property "Rating" "4.7A"
+			(at 156.21 134.62 0)
+			(hide yes)
+			(show_name no)
+			(do_not_autoplace no)
+			(effects
+				(font
+					(size 1.27 1.27)
+				)
+			)
+		)
+		(property "Id" "PowerSwitch:${SYMBOL_NAME}"
+			(at 156.21 125.73 0)
+			(hide yes)
+			(show_name no)
+			(do_not_autoplace no)
+			(effects
+				(font
+					(size 1.27 1.27)
+				)
+			)
+		)
+		(property "Sim.Pin" ""
+			(at 156.21 106.68 0)
+			(hide yes)
+			(show_name no)
+			(do_not_autoplace no)
+			(effects
+				(font
+					(size 1.27 1.27)
+				)
+			)
+		)
+		(property "Voltage" ""
+			(at 156.21 106.68 0)
+			(hide yes)
+			(show_name no)
+			(do_not_autoplace no)
+			(effects
+				(font
+					(size 1.27 1.27)
+				)
+			)
+		)
 		(pin "1"
 		)
@@
 			)
 		)
+		(property "Id" "Resistor:${SYMBOL_NAME}"
+			(at 121.92 114.3 0)
+			(hide yes)
+			(show_name no)
+			(do_not_autoplace no)
+			(effects
+				(font
+					(size 1.27 1.27)
+				)
+			)
+		)
+		(property "Sim.Pin" ""
+			(at 135.89 114.3 90)
+			(hide yes)
+			(show_name no)
+			(do_not_autoplace no)
+			(effects
+				(font
+					(size 1.27 1.27)
+				)
+			)
+		)
+		(property "Voltage" ""
+			(at 135.89 114.3 90)
+			(hide yes)
+			(show_name no)
+			(do_not_autoplace no)
+			(effects
+				(font
+					(size 1.27 1.27)
+				)
+			)
+		)
 		(pin "1"
 		)
@@
 		(dnp no)
 		(fields_autoplaced yes)
-		(property "Reference" "#PWR703"
+		(property "Reference" "#PWR0703"
 			(at 172.72 114.3 0)
 			(hide yes)
@@
 			(project "beat"
 				(path "/6c8448b4-b04d-47e1-934e-e40cbe27a7be/0ac9d349-3066-4d6a-93e7-4d57eaae463a"
-					(reference "#PWR703")
+					(reference "#PWR0703")
 					(unit 1)
 				)
