File: hardware/PowerSwitch.kicad_sch (KiCad schematic)
At the start: 2 parts, among them U701 TPS2559

Commit message: Good Bye Imperial
Parts:
- R701: footprint V2_Resistor_SMD:R_0603 -> V2_Resistor_SMD:R_1608; symbol V2_Resistor:0603_39k -> V2_Resistor:1608_39k
Changed lines of the file:
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@@
 	)
 	(symbol
-		(lib_id "V2_Resistor:0603_39k")
+		(lib_id "V2_Resistor:1608_39k")
 		(at 135.89 114.3 270)
 		(unit 1)
@@
 			)
 		)
-		(property "Footprint" "V2_Resistor_SMD:R_0603"
+		(property "Footprint" "V2_Resistor_SMD:R_1608"
 			(at 120.142 114.3 0)
 			(hide yes)
