File: hardware/PWMChannel.kicad_sch (KiCad schematic)
At the start: 4 parts, among them Q201 IQE006NE2LM5CG

Commit message: Update
Parts:
- C201: Id (none) -> Capacitor:${SYMBOL_NAME}
- D201: Id (none) -> Diode:${SYMBOL_NAME}
- D202: Id (none) -> LED:${SYMBOL_NAME}; Rating (none) -> 15mA
- Q201: Id (none) -> MOSFET:${SYMBOL_NAME}
Other:
- company: Power MOSFET + RGB LED -> Versio Duo
Changed lines of the file:
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@@
 	(title_block
 		(title "V2 beat")
-		(date "2026-03-30")
+		(date "2026-04-14")
 		(rev "2026-03-30")
-		(company "Power MOSFET + RGB LED")
+		(company "Versio Duo")
+		(comment 1 "Solenoid Controller")
 	)
 	(junction
@@
 			)
 		)
+		(property "Id" "Diode:${SYMBOL_NAME}"
+			(at 134.62 88.9 0)
+			(hide yes)
+			(show_name no)
+			(do_not_autoplace no)
+			(effects
+				(font
+					(size 1.27 1.27)
+				)
+			)
+		)
+		(property "Sim.Pin" ""
+			(at 146.05 88.9 90)
+			(hide yes)
+			(show_name no)
+			(do_not_autoplace no)
+			(effects
+				(font
+					(size 1.27 1.27)
+				)
+			)
+		)
+		(property "Voltage" ""
+			(at 146.05 88.9 90)
+			(hide yes)
+			(show_name no)
+			(do_not_autoplace no)
+			(effects
+				(font
+					(size 1.27 1.27)
+				)
+			)
+		)
 		(pin "1"
 		)
@@
 			)
 		)
+		(property "Id" "Capacitor:${SYMBOL_NAME}"
+			(at 133.35 104.14 0)
+			(hide yes)
+			(show_name no)
+			(do_not_autoplace no)
+			(effects
+				(font
+					(size 1.27 1.27)
+				)
+			)
+		)
+		(property "Sim.Pin" ""
+			(at 133.35 88.9 0)
+			(hide yes)
+			(show_name no)
+			(do_not_autoplace no)
+			(effects
+				(font
+					(size 1.27 1.27)
+				)
+			)
+		)
+		(property "Voltage" ""
+			(at 133.35 88.9 0)
+			(hide yes)
+			(show_name no)
+			(do_not_autoplace no)
+			(effects
+				(font
+					(size 1.27 1.27)
+				)
+			)
+		)
 		(pin "1"
 		)
@@
 			)
 		)
+		(property "Id" "MOSFET:${SYMBOL_NAME}"
+			(at 130.81 110.49 0)
+			(hide yes)
+			(show_name no)
+			(do_not_autoplace no)
+			(effects
+				(font
+					(size 1.27 1.27)
+				)
+			)
+		)
+		(property "Sim.Pin" ""
+			(at 130.81 96.52 0)
+			(hide yes)
+			(show_name no)
+			(do_not_autoplace no)
+			(effects
+				(font
+					(size 1.27 1.27)
+				)
+			)
+		)
+		(property "Voltage" ""
+			(at 130.81 96.52 0)
+			(hide yes)
+			(show_name no)
+			(do_not_autoplace no)
+			(effects
+				(font
+					(size 1.27 1.27)
+				)
+			)
+		)
 		(pin "1"
 		)
@@
 		(in_pos_files yes)
 		(dnp no)
-		(property "Reference" "#PWR203"
+		(property "Reference" "#PWR0203"
 			(at 166.37 127 0)
 			(hide yes)
@@
 			(project "beat"
 				(path "/6c8448b4-b04d-47e1-934e-e40cbe27a7be/20fe3b49-6fc0-49b3-882e-b60ec2c37622"
-					(reference "#PWR403")
+					(reference "#PWR0403")
 					(unit 1)
 				)
 				(path "/6c8448b4-b04d-47e1-934e-e40cbe27a7be/6b0ff6e6-8459-48b3-ad82-b75391ec7027"
-					(reference "#PWR203")
+					(reference "#PWR0203")
 					(unit 1)
 				)
 				(path "/6c8448b4-b04d-47e1-934e-e40cbe27a7be/d14b4538-8a69-4c12-9312-e76942186e04"
-					(reference "#PWR503")
+					(reference "#PWR0503")
 					(unit 1)
 				)
 				(path "/6c8448b4-b04d-47e1-934e-e40cbe27a7be/e8fd4e45-6455-499e-826d-b4439d3dc293"
-					(reference "#PWR303")
+					(reference "#PWR0303")
 					(unit 1)
 				)
@@
 			)
 		)
+		(property "Id" "LED:${SYMBOL_NAME}"
+			(at 152.4 134.62 0)
+			(hide yes)
+			(show_name no)
+			(do_not_autoplace no)
+			(effects
+				(font
+					(size 1.27 1.27)
+				)
+			)
+		)
+		(property "Rating" "15mA"
+			(at 152.4 149.86 0)
+			(hide yes)
+			(show_name no)
+			(do_not_autoplace no)
+			(effects
+				(font
+					(size 1.27 1.27)
+				)
+			)
+		)
+		(property "Sim.Pin" ""
+			(at 152.4 125.73 0)
+			(hide yes)
+			(show_name no)
+			(do_not_autoplace no)
+			(effects
+				(font
+					(size 1.27 1.27)
+				)
+			)
+		)
+		(property "Voltage" ""
+			(at 152.4 125.73 0)
+			(hide yes)
+			(show_name no)
+			(do_not_autoplace no)
+			(effects
+				(font
+					(size 1.27 1.27)
+				)
+			)
+		)
 		(pin "1"
 		)
@@
 		(in_pos_files yes)
 		(dnp no)
-		(property "Reference" "#PWR201"
+		(property "Reference" "#PWR0201"
 			(at 133.35 107.95 0)
 			(hide yes)
@@
 			(project "beat"
 				(path "/6c8448b4-b04d-47e1-934e-e40cbe27a7be/20fe3b49-6fc0-49b3-882e-b60ec2c37622"
-					(reference "#PWR401")
+					(reference "#PWR0401")
 					(unit 1)
 				)
 				(path "/6c8448b4-b04d-47e1-934e-e40cbe27a7be/6b0ff6e6-8459-48b3-ad82-b75391ec7027"
-					(reference "#PWR201")
+					(reference "#PWR0201")
 					(unit 1)
 				)
 				(path "/6c8448b4-b04d-47e1-934e-e40cbe27a7be/d14b4538-8a69-4c12-9312-e76942186e04"
-					(reference "#PWR501")
+					(reference "#PWR0501")
 					(unit 1)
 				)
 				(path "/6c8448b4-b04d-47e1-934e-e40cbe27a7be/e8fd4e45-6455-499e-826d-b4439d3dc293"
-					(reference "#PWR301")
+					(reference "#PWR0301")
 					(unit 1)
 				)
@@
 		(in_pos_files yes)
 		(dnp no)
-		(property "Reference" "#PWR202"
+		(property "Reference" "#PWR0202"
 			(at 156.21 121.92 0)
 			(hide yes)
@@
 			(project "beat"
 				(path "/6c8448b4-b04d-47e1-934e-e40cbe27a7be/20fe3b49-6fc0-49b3-882e-b60ec2c37622"
-					(reference "#PWR402")
+					(reference "#PWR0402")
 					(unit 1)
 				)
 				(path "/6c8448b4-b04d-47e1-934e-e40cbe27a7be/6b0ff6e6-8459-48b3-ad82-b75391ec7027"
-					(reference "#PWR202")
+					(reference "#PWR0202")
 					(unit 1)
 				)
 				(path "/6c8448b4-b04d-47e1-934e-e40cbe27a7be/d14b4538-8a69-4c12-9312-e76942186e04"
-					(reference "#PWR502")
+					(reference "#PWR0502")
 					(unit 1)
 				)
 				(path "/6c8448b4-b04d-47e1-934e-e40cbe27a7be/e8fd4e45-6455-499e-826d-b4439d3dc293"
-					(reference "#PWR302")
-					(unit 1)
-				)
+					(reference "#PWR0302")
+					(unit 1)
+				)

Commit message: Good Bye Imperial
Parts:
- C201: footprint V2_Capacitor_SMD:C_0603 -> V2_Capacitor_SMD:C_1608; symbol V2_Capacitor:0603_0u1 -> V2_Capacitor:1608_0u1
Changed lines of the file:
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@@
 	)
 	(symbol
-		(lib_id "V2_Capacitor:0603_0u1")
+		(lib_id "V2_Capacitor:1608_0u1")
 		(at 133.35 88.9 0)
 		(unit 1)
@@
 			)
 		)
-		(property "Footprint" "V2_Capacitor_SMD:C_0603"
+		(property "Footprint" "V2_Capacitor_SMD:C_1608"
 			(at 133.35 105.918 0)
 			(hide yes)
