File: hardware/PWMChannel.kicad_sch (KiCad schematic)
At the start: 4 parts, among them Q201 IQE006NE2LM5CG

Commit message: Refresh
Connections:
- net PWMOut renamed PWM-Sink
- net Power renamed +VPWM
Changed lines of the file:
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@@
 	(title_block
 		(title "V2 beat")
-		(date "2026-08-19")
+		(date "2026-08-28")
 		(rev "2026-08-19")
 		(company "Versio Duo")
@@
 		)
 	)
-	(hierarchical_label "PWMOut"
+	(hierarchical_label "PWM-Sink"
 		(shape output)
 		(at 185.42 91.44 0)
@@
 		)
 	)
-	(hierarchical_label "Power"
+	(hierarchical_label "+VPWM"
 		(shape input)
 		(at 121.92 86.36 180)
@@
 		(in_pos_files yes)
 		(dnp no)
-		(property "Reference" "#PWR0203"
+		(property "Reference" "#PWR203"
 			(at 166.37 127 0)
 			(hide yes)
@@
 			(project "beat"
 				(path "/6c8448b4-b04d-47e1-934e-e40cbe27a7be/20fe3b49-6fc0-49b3-882e-b60ec2c37622"
-					(reference "#PWR0403")
+					(reference "#PWR403")
 					(unit 1)
 				)
 				(path "/6c8448b4-b04d-47e1-934e-e40cbe27a7be/6b0ff6e6-8459-48b3-ad82-b75391ec7027"
-					(reference "#PWR0203")
+					(reference "#PWR203")
 					(unit 1)
 				)
 				(path "/6c8448b4-b04d-47e1-934e-e40cbe27a7be/d14b4538-8a69-4c12-9312-e76942186e04"
-					(reference "#PWR0503")
+					(reference "#PWR503")
 					(unit 1)
 				)
 				(path "/6c8448b4-b04d-47e1-934e-e40cbe27a7be/e8fd4e45-6455-499e-826d-b4439d3dc293"
-					(reference "#PWR0303")
+					(reference "#PWR303")
 					(unit 1)
 				)
@@
 		(in_pos_files yes)
 		(dnp no)
-		(property "Reference" "#PWR0201"
+		(property "Reference" "#PWR201"
 			(at 133.35 107.95 0)
 			(hide yes)
@@
 			(project "beat"
 				(path "/6c8448b4-b04d-47e1-934e-e40cbe27a7be/20fe3b49-6fc0-49b3-882e-b60ec2c37622"
-					(reference "#PWR0401")
+					(reference "#PWR401")
 					(unit 1)
 				)
 				(path "/6c8448b4-b04d-47e1-934e-e40cbe27a7be/6b0ff6e6-8459-48b3-ad82-b75391ec7027"
-					(reference "#PWR0201")
+					(reference "#PWR201")
 					(unit 1)
 				)
 				(path "/6c8448b4-b04d-47e1-934e-e40cbe27a7be/d14b4538-8a69-4c12-9312-e76942186e04"
-					(reference "#PWR0501")
+					(reference "#PWR501")
 					(unit 1)
 				)
 				(path "/6c8448b4-b04d-47e1-934e-e40cbe27a7be/e8fd4e45-6455-499e-826d-b4439d3dc293"
-					(reference "#PWR0301")
+					(reference "#PWR301")
 					(unit 1)
 				)
@@
 		(in_pos_files yes)
 		(dnp no)
-		(property "Reference" "#PWR0202"
+		(property "Reference" "#PWR202"
 			(at 156.21 121.92 0)
 			(hide yes)
@@
 			(project "beat"
 				(path "/6c8448b4-b04d-47e1-934e-e40cbe27a7be/20fe3b49-6fc0-49b3-882e-b60ec2c37622"
-					(reference "#PWR0402")
+					(reference "#PWR402")
 					(unit 1)
 				)
 				(path "/6c8448b4-b04d-47e1-934e-e40cbe27a7be/6b0ff6e6-8459-48b3-ad82-b75391ec7027"
-					(reference "#PWR0202")
+					(reference "#PWR202")
 					(unit 1)
 				)
 				(path "/6c8448b4-b04d-47e1-934e-e40cbe27a7be/d14b4538-8a69-4c12-9312-e76942186e04"
-					(reference "#PWR0502")
+					(reference "#PWR502")
 					(unit 1)
 				)
 				(path "/6c8448b4-b04d-47e1-934e-e40cbe27a7be/e8fd4e45-6455-499e-826d-b4439d3dc293"
-					(reference "#PWR0302")
-					(unit 1)
-				)
+					(reference "#PWR302")
+					(unit 1)
+				)
