File: hardware/beat-cover-camp/beat-cover-camp.kicad_pcb (KiCad board)
At the start: 2 copper layers, 60 x 35 mm, 11 parts

Commit message: Replace Order_Number
Parts:
- H101, H102, H103, H104: value MountingHole_2mm_Pad_5.2mm -> 2mm_Pad_5.2mm; footprint V2_Mechanical:Mounting_Hole_2mm_Pad_5.2mm -> V2_Mechanical:MountingHole_2mm_Pad_5.2mm
- H105: value MountingHole_1mm -> 1mm
- H106, H107, H108, H109: value Mounting_Hole -> 2mm_Pad_2.4mm
- INFO101: value ORDER-NUMBER -> ~; footprint V2_Production:Order_Number -> V2_Production:Revision
